File: board_v1/Board_v1.brd (EAGLE design)
At the start: 135.1 x 89 mm, 19 parts, among them IC1 MAX7219, IC2 MAX7219, IC3 MAX7219

Commit message: PCB v1 WIP
Parts:
- removed U$1: MRB_ROTARY_SWITCH, AES_lib:MRB24B_SP3T
- added 12VIN: CONN3, AES_lib:MICRO-FIT_43560_3MM
- added BTN: CONN1, AES_lib:MICRO-FIT_43560_3MM
- added C1, C2, C3: 10uF, AES_lib:CPOL-RADIAL-2.5MM-5MM-KIT
- added C4, C5, C6: 100nF, AES_lib:CAP-PTH-5MM
- added D1: 1N4001, AES_lib:CASE59−10-AXIAL
- added MOSFET: IRLB872, AES_lib:TO-220-ALT
- added R1: 28k, AES_lib:AXIAL-0.3
- added R2, R3: 23k, AES_lib:AXIAL-0.3
- added R4: 10k, AES_lib:AXIAL-0.3
- added SOUT: CONN2, AES_lib:MICRO-FIT_43560_3MM
- added SW1: ROTARY SWITCH, AES_lib:MRB24B_SP3T
- added VREG: L7805CV, AES_lib:TO-220-ALT
- CONV: value 3-5V_LOGIC_LVL_CONV -> LOGIC LVL CONV
- moved IC3 51.4 mm to (16.9, -14.5), turned to 90 degrees
- moved CONV 26.6 mm to (42.7, 9.30), turned to 270 degrees
- moved IC2 6.32 mm to (68.9, 20.6)
- moved SEV1 3.28 mm to (-28.9, 14.6)
- moved SEV2 3.28 mm to (-21.3, 14.6)
- moved SEV3 2.84 mm to (-3.75, 23.4)
- moved SEV4 2.82 mm to (3.84, 23.4)
- moved SEV6 2.44 mm to (29.3, 14.6)
- moved SEV5 2.43 mm to (21.7, 14.6)
- moved FEATHERM0 1.55 mm to (87.0, -22.8)
- moved SEV7 0.48 mm to (-42.1, -36.5)
- moved SEV9 0.48 mm to (-26.8, -36.5)
- moved SEV10 0.47 mm to (-19.2, -36.5)
- moved SEV8 0.47 mm to (-34.5, -36.5)
Connections:
- removed net VCC: IC1.19, IC2.19, IC3.19
- new net 12V: 12VIN.P$2, D1.CAT, SOUT.P$2, VREG.IN
- new net 3.3V: FEATHERM0.2
- new net 5V: FEATHERM0.26, IC1.19, IC2.19, IC3.19, R1.P$1, R2.P$1, R3.P$1, VREG.OUT
- new net N$1: IC1.18, R1.P$2
- new net N$10: IC1.13, IC2.13, IC3.13
- new net N$11: IC1.12, IC2.12, IC3.12
- new net N$12: IC1.1
- new net N$13: IC1.24, IC3.1
- new net N$14: IC2.1, IC3.24
- new net N$2: D1.ANOD, MOSFET.GND, SOUT.P$1
- new net N$3: MOSFET.IN
- new net N$4: SW1.1
- new net N$5: SW1.2
- new net N$6: SW1.3
- new net N$7: R4.P$2, SW1.C1
- new net N$8: IC2.18, R3.P$2
- new net N$9: IC3.18, R2.P$2
- net GND: now also 12VIN.P$1, CONV.GND, CONV.GND2, MOSFET.OUT, R4.P$1, VREG.GND

Commit message: added button pcb
Parts:
- added R5: 10k, AES_lib:AXIAL-0.3
- moved FEATHERM0 1.35 mm to (87.0, -21.5)
- moved CONV 1.15 mm to (43.0, 10.4), flipped to the bottom
Connections:
- new net N$16: BTN.P$2
- net 3.3V: now also BTN.P$1, R5.P$2
- net GND: now also R5.P$1
Other:
- outline, holes or cut-outs redrawn

Commit message: ready to start routing?
Parts:
- added J1: (no value), SparkFun-Connectors:1X04_NO_SILK
- added R6: 10k, AES_lib:AXIAL-0.3
- C2: value 10uF -> 100nF; device AES_lib:CPOL-RADIAL-2.5MM-5MM-KIT -> AES_lib:CAP-PTH-5MM
- C5: value 100nF -> 10uF; device AES_lib:CAP-PTH-5MM -> AES_lib:CPOL-RADIAL-2.5MM-5MM-KIT
- R2: value 23k -> 28k
- moved R5 106.5 mm to (61.0, -24.5)
- moved R3 106.2 mm to (24.5, -38.0), turned to 90 degrees
- moved R4 105.0 mm to (0.00, 2.50), turned to 180 degrees
- moved C6 91.5 mm to (24.0, -19.5), turned to 90 degrees
- moved C5 90.7 mm to (24.5, -29.0), turned to 90 degrees
- moved C4 89.1 mm to (31.0, -14.5), turned to 90 degrees
- moved R2 83.5 mm to (39.0, -6.00), turned to 90 degrees
- moved C3 75.7 mm to (31.0, -5.50), turned to 90 degrees
- moved R1 66.5 mm to (53.5, 39.5), turned to 180 degrees
- moved C1 48.1 mm to (63.5, 39.5), turned to 180 degrees
- moved VREG 42.5 mm to (-15.7, -19.7), turned to 0 degrees
- moved CONV 35.1 mm to (78.0, 13.4), turned to 0 degrees
- moved C2 30.7 mm to (71.5, 39.5)
- moved IC2 17.9 mm to (52.4, 13.5), turned to 180 degrees
- moved MOSFET 16.7 mm to (-42.6, 1.00), turned to 270 degrees
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Connections:
- removed net N$10: IC1.13, IC2.13, IC3.13
- removed net N$11: IC1.12, IC2.12, IC3.12
- removed net N$12: IC1.1
- removed net N$16: BTN.P$2
- removed net N$4: SW1.1
- removed net N$5: SW1.2
- removed net N$6: SW1.3
- new net BTN: BTN.P$2, FEATHERM0.21
- new net CLK: CONV.1, IC1.13, IC2.13, IC3.13
- new net CLK3: CONV.7, FEATHERM0.24
- new net DIG01: BAR2.1, IC1.2
- new net DIG02: BAR1.1, IC2.2
- new net DIG03: IC3.2, SEV7.1, SEV7.6
- new net DIG11: BAR2.6, IC1.11
- new net DIG12: BAR1.6, IC2.11
- new net DIG13: IC3.11, SEV8.1, SEV8.6
- new net DIG21: BAR2.7, IC1.6
- new net DIG22: BAR1.7, IC2.6
- new net DIG23: IC3.6, SEV9.1, SEV9.6
- new net DIG31: BAR3.1, IC1.7
- new net DIG32: IC2.7, SEV1.1, SEV1.6
- new net DIG33: IC3.7, SEV10.1, SEV10.6
- new net DIG41: BAR3.6, IC1.3
- new net DIG42: IC2.3, SEV2.1, SEV2.6
- new net DIG43: IC3.3, SEV5.1, SEV5.6
- new net DIG51: BAR3.7, IC1.10
- new net DIG52: IC2.10, SEV3.1, SEV3.6
- new net DIG53: IC3.10, SEV6.1, SEV6.6
- new net DIG62: IC2.5, SEV4.1, SEV4.6
- new net DIN: CONV.5, IC1.1
- new net DIN3: CONV.11, FEATHERM0.22
- new net LOAD: CONV.2, IC1.12, IC2.12, IC3.12
- new net LOAD3: CONV.8, FEATHERM0.23
- new net RESET: FEATHERM0.1, J1.2
- new net S1: FEATHERM0.20, SW1.1
- new net S2: FEATHERM0.19, SW1.2
- new net S3: FEATHERM0.18, SW1.3
- new net SEGA1: BAR2.2, BAR3.2, IC1.14
- new net SEGA2: BAR1.2, IC2.14, SEV1.10, SEV2.10, SEV3.10, SEV4.10
- new net SEGA3: IC3.14, SEV10.10, SEV5.10, SEV6.10, SEV7.10, SEV8.10, SEV9.10
- new net SEGB1: BAR2.13, BAR3.13, IC1.16
- new net SEGB2: BAR1.13, IC2.16, SEV1.9, SEV2.9, SEV3.9, SEV4.9
- new net SEGB3: IC3.16, SEV10.9, SEV5.9, SEV6.9, SEV7.9, SEV8.9, SEV9.9
- new net SEGC1: BAR2.3, BAR3.3, IC1.20
- new net SEGC2: BAR1.3, IC2.20, SEV1.8, SEV2.8, SEV3.8, SEV4.8
- new net SEGC3: IC3.20, SEV10.8, SEV5.8, SEV6.8, SEV7.8, SEV8.8, SEV9.8
- new net SEGD1: BAR2.12, BAR3.12, IC1.23
- new net SEGD2: BAR1.12, IC2.23, SEV1.5, SEV2.5, SEV3.5, SEV4.5
- new net SEGD3: IC3.23, SEV10.5, SEV5.5, SEV6.5, SEV7.5, SEV8.5, SEV9.5
- new net SEGDP1: BAR2.10, BAR3.10, IC1.22
- new net SEGDP2: BAR1.10, IC2.22, SEV1.7, SEV2.7, SEV3.7, SEV4.7
- new net SEGDP3: IC3.22, SEV10.7, SEV5.7, SEV6.7, SEV7.7, SEV8.7, SEV9.7
- new net SEGE1: BAR2.4, BAR3.4, IC1.21
- new net SEGE2: BAR1.4, IC2.21, SEV1.4, SEV2.4, SEV3.4, SEV4.4
- new net SEGE3: IC3.21, SEV10.4, SEV5.4, SEV6.4, SEV7.4, SEV8.4, SEV9.4
- new net SEGF1: BAR2.11, BAR3.11, IC1.15
- new net SEGF2: BAR1.11, IC2.15, SEV1.2, SEV2.2, SEV3.2, SEV4.2
- new net SEGF3: IC3.15, SEV10.2, SEV5.2, SEV6.2, SEV7.2, SEV8.2, SEV9.2
- new net SEGG1: BAR2.5, BAR3.5, IC1.17
- new net SEGG2: BAR1.5, IC2.17, SEV1.3, SEV2.3, SEV3.3, SEV4.3
- new net SEGG3: IC3.17, SEV10.3, SEV5.3, SEV6.3, SEV7.3, SEV8.3, SEV9.3
- new net STA: FEATHERM0.17, J1.3
- net 3.3V: now also CONV.9, J1.4, R6.P$2
- net 5V: now also C1.1, C2.1, C3.1, C4.1, C5.1, C6.1, CONV.3
- net GND: now also C1.2, C2.2, C3.2, C4.2, C5.2, C6.2, J1.1, R6.P$1
- net N$13: now also IC2.1; no longer IC3.1
- net N$14: now also IC2.24, IC3.1; no longer IC2.1, IC3.24
- net N$3: now also CONV.6
- net N$8: now also IC3.18; no longer IC2.18
- net N$9: now also IC2.18; no longer IC3.18

Commit message: routing v1 finish
Parts:
- moved R2 29.1 mm to (43.8, 22.7), turned to 0 degrees
- moved R1 19.0 mm to (72.5, 39.5), turned to 0 degrees
- moved C1 9.40 mm to (54.1, 39.5), turned to 0 degrees
- moved C2 9.40 mm to (62.1, 39.5)
- moved SEV9 7.62 mm to (-26.9, -36.5)
- moved SEV10 7.62 mm to (-19.2, -36.5)
- moved C3 3.82 mm to (31.3, -9.31)
- moved C4 2.55 mm to (31.3, -17.0)
- moved IC1 1.02 mm to (66.5, 28.6)
- moved C5 0.51 mm to (24.0, -29.0)
- moved R3 0.51 mm to (24.0, -38.0)
- moved IC3 0.25 mm to (14.7, -27.9), turned to 90 degrees
- turned IC2 to 0 degrees
Connections:
- net SEGDP2: no longer SEV1.7, SEV2.7, SEV3.7, SEV4.7
- net SEGDP3: no longer SEV10.7, SEV5.7, SEV8.7
Routing:
- net SEGF2: track 0.00 -> 153.2 mm, vias 0 -> 1
- net SEGB2: track 0.00 -> 140.8 mm, vias 0 -> 3
- net SEGG2: track 0.00 -> 138.1 mm, vias 0 -> 4
- net SEGD2: track 0.00 -> 137.1 mm, vias 0 -> 4
- net SEGE2: track 0.00 -> 132.3 mm, vias 0 -> 2
- net SEGE3: track 0.00 -> 126.9 mm, vias 0 -> 1
- net SEGC2: track 0.00 -> 123.7 mm, vias 0 -> 2
- net SEGA2: track 0.00 -> 123.6 mm
- net SEGD3: track 0.00 -> 123.3 mm
- net SEGC3: track 0.00 -> 122.5 mm, vias 0 -> 1
- net N$3: track 0.00 -> 121.5 mm, vias 0 -> 2
- net SEGDP3: track 0.00 -> 120.1 mm, vias 0 -> 1
- net SEGA3: track 0.00 -> 119.5 mm, vias 0 -> 1
- net SEGF3: track 0.00 -> 117.3 mm, vias 0 -> 1
- net SEGB3: track 0.00 -> 116.9 mm, vias 0 -> 2
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- added copper zone on layer 1, net 5V
- added copper zone on layer 16, net GND
Other:
- outline, holes or cut-outs redrawn

Commit message: ready for fabhouse v1
Routing:
- net SEGA3: track 119.5 -> 117.0 mm
- net STA: track 49.7 -> 51.6 mm
- net SEGG3: track 115.2 -> 117.0 mm
- net SEGD2: track 137.1 -> 135.8 mm
- net SEGDP3: track 120.1 -> 121.1 mm
- net SEGC2: track 123.7 -> 123.2 mm
Other:
- board text added: "12V IN"
- board text added: "BTN"
- board text added: "KETTLE META-CONTROLLER rev1. Jan-2019 Design Informatics"
- board text added: "SOLENOID"
