File: button_pcb_v1/button_pcb_v1.brd (EAGLE design)
At the start: 22.5 x 21 mm, 2 parts

Commit message: ready for fabhouse v1
Parts:
- moved J1 0.76 mm to (-1.22, 7.20)
Routing:
- net N$2: track 10.8 -> 11.6 mm
- net N$1: track 14.1 -> 14.9 mm, vias 0 -> 1
- added copper zone on layer 16, net N$4
Other:
- board size 22.5 x 21 mm -> 22.5 x 21.5 mm
Changed lines of the file:
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@@
 </layers>
 <board>
-<fusionsync huburn="a.cGVyc29uYWw6dWUyOWQyYjdi" projecturn="a.cGVyc29uYWw6dWUyOWQyYjdiIzIwMTgxMTMwMTYzMTgyOTAx" f3durn="urn:adsk.wipprod:dm.lineage:K_lnejlhTFO0_kCaxYINUQ" pcbguid="7cc0ec74-97cc-4953-9a47-41e4ec11a13e" lastpulledtime="2018-12-12T10:51:54Z" lastsyncedchangeguid="be66b80d-e6ea-1d77-c099-e3a73e79f2f7"/>
+<fusionsync huburn="a.cGVyc29uYWw6dWUyOWQyYjdi" projecturn="a.cGVyc29uYWw6dWUyOWQyYjdiIzIwMTgxMTMwMTYzMTgyOTAx" f3durn="urn:adsk.wipprod:dm.lineage:K_lnejlhTFO0_kCaxYINUQ" pcbguid="7cc0ec74-97cc-4953-9a47-41e4ec11a13e" lastpulledtime="2018-12-12T10:51:54Z" lastsyncedchangeguid="efa3357b-d71f-c06c-1bd3-ce90f2470ee8"/>
 <plain>
 <hole x="-7.15" y="6.4" drill="3.2"/>
 <hole x="7.15" y="6.4" drill="3.2"/>
-<wire x1="-11.25" y1="-10.5" x2="11.25" y2="-10.5" width="0.254" layer="20"/>
-<wire x1="11.25" y1="-10.5" x2="11.25" y2="10.5" width="0.254" layer="20"/>
-<wire x1="11.25" y1="10.5" x2="-11.25" y2="10.5" width="0.254" layer="20"/>
-<wire x1="-11.25" y1="10.5" x2="-11.25" y2="-10.5" width="0.254" layer="20"/>
+<wire x1="11.249996875" y1="-8.465425" x2="11.2269125" y2="9.25794375" width="0.254" layer="20"/>
+<wire x1="11.2269125" y1="9.25794375" x2="9.448915625" y2="11.0334" width="0.254" layer="20" curve="89.925279"/>
+<wire x1="9.448915625" y1="11.0334" x2="-9.49508125" y2="11.0334" width="0.254" layer="20"/>
+<wire x1="-9.49508125" y1="11.0334" x2="-11.27308125" y2="9.253146875" width="0.254" layer="20" curve="90.072607"/>
+<wire x1="-11.27308125" y1="9.253146875" x2="-11.249996875" y2="-8.470221875" width="0.254" layer="20"/>
+<wire x1="-11.249996875" y1="-8.470221875" x2="-9.217996875" y2="-10.5" width="0.254" layer="20" curve="89.925455"/>
+<wire x1="-9.217996875" y1="-10.5" x2="9.218" y2="-10.5" width="0.254" layer="20"/>
+<wire x1="9.218" y1="-10.5" x2="11.249996875" y2="-8.465425" width="0.254" layer="20" curve="90.072607"/>
 </plain>
 <attributes>
@@
 <param name="mtCopper" value="0.035mm 0.035mm 0.035mm 0.035mm 0.035mm 0.035mm 0.035mm 0.035mm 0.035mm 0.035mm 0.035mm 0.035mm 0.035mm 0.035mm 0.035mm 0.035mm"/>
 <param name="mtIsolate" value="1.5mm 0.15mm 0.2mm 0.15mm 0.2mm 0.15mm 0.2mm 0.15mm 0.2mm 0.15mm 0.2mm 0.15mm 0.2mm 0.15mm 0.2mm"/>
-<param name="mdWireWire" value="6mil"/>
-<param name="mdWirePad" value="6mil"/>
-<param name="mdWireVia" value="6mil"/>
-<param name="mdPadPad" value="6mil"/>
-<param name="mdPadVia" value="6mil"/>
-<param name="mdViaVia" value="6mil"/>
+<param name="mdWireWire" value="8mil"/>
+<param name="mdWirePad" value="8mil"/>
+<param name="mdWireVia" value="8mil"/>
+<param name="mdPadPad" value="8mil"/>
+<param name="mdPadVia" value="8mil"/>
+<param name="mdViaVia" value="8mil"/>
 <param name="mdSmdPad" value="6mil"/>
 <param name="mdSmdVia" value="6mil"/>
@@
 <attribute name="NAME" x="0" y="-2.99" size="1.016" layer="25" font="vector" ratio="12" align="bottom-center"/>
 </element>
-<element name="J1" library="SparkFun-Connectors" library_urn="urn:adsk.eagle:library:513" package="1X02_NO_SILK" package3d_urn="urn:adsk.eagle:package:38051/1" value="" x="-1.216" y="6.44" smashed="yes">
-<attribute name="VALUE" x="-2.486" y="4.408" size="0.6096" layer="27" font="vector" ratio="20"/>
+<element name="J1" library="SparkFun-Connectors" library_urn="urn:adsk.eagle:library:513" package="1X02_NO_SILK" package3d_urn="urn:adsk.eagle:package:38051/1" value="" x="-1.216" y="7.202" smashed="yes">
+<attribute name="VALUE" x="-2.486" y="5.17" size="0.6096" layer="27" font="vector" ratio="20"/>
 </element>
 </elements>
@@
 <contactref element="BTN" pad="3"/>
 <contactref element="BTN" pad="2"/>
-<wire x1="6.35" y1="-5.57" x2="1.3208" y2="-0.5408" width="0.381" layer="1"/>
-<wire x1="1.3208" y1="6.4368" x2="1.324" y2="6.44" width="0.381" layer="1"/>
-<wire x1="1.3208" y1="-0.5408" x2="1.3208" y2="6.4368" width="0.381" layer="1"/>
-<wire x1="1.3208" y1="-0.5408" x2="-6.35" y2="-5.57" width="0" layer="19" extent="1-1"/>
+<wire x1="6.35" y1="-5.57" x2="1.3208" y2="-0.5408" width="0.381" layer="16"/>
+<wire x1="1.3208" y1="7.1988" x2="1.324" y2="7.202" width="0.381" layer="1"/>
+<wire x1="1.3208" y1="-0.5408" x2="1.3208" y2="7.1988" width="0.381" layer="16"/>
+<via x="1.3208" y="7.1988" extent="1-16" drill="0.35"/>
+<wire x1="1.3208" y1="-0.5408" x2="-6.35" y2="-5.57" width="0" layer="19" extent="16-16"/>
 </signal>
 <signal name="N$2">
@@
 <contactref element="BTN" pad="1"/>
 <contactref element="BTN" pad="4"/>
-<wire x1="-6.35" y1="-0.49" x2="-3.3348" y2="-0.49" width="0.381" layer="1"/>
-<wire x1="-1.216" y1="1.6288" x2="-1.216" y2="6.44" width="0.381" layer="1"/>
-<wire x1="-3.3348" y1="-0.49" x2="-1.216" y2="1.6288" width="0.381" layer="1"/>
-<wire x1="-1.216" y1="1.6288" x2="6.35" y2="-0.49" width="0" layer="19" extent="1-1"/>
+<wire x1="-6.35" y1="-0.49" x2="-3.3348" y2="-0.49" width="0.381" layer="16"/>
+<wire x1="-1.216" y1="1.6288" x2="-1.216" y2="7.202" width="0.381" layer="16"/>
+<wire x1="-3.3348" y1="-0.49" x2="-1.216" y2="1.6288" width="0.381" layer="16"/>
+<wire x1="-1.216" y1="1.6288" x2="6.35" y2="-0.49" width="0" layer="19" extent="16-16"/>
 </signal>
 <signal name="GND">
-<polygon width="0.254" layer="1" isolate="0.3048">
-<vertex x="-11.25" y="10.5"/>
+<polygon width="0.254" layer="1" isolate="0.381">
+<vertex x="11.25" y="11.262"/>
+<vertex x="-11.25" y="11.262"/>
 <vertex x="-11.25" y="-10.5"/>
 <vertex x="11.25" y="-10.5"/>
-<vertex x="11.25" y="10.5"/>
 </polygon>
-</signal>
+<polygon width="0.254" layer="1" isolate="0.3048">
+<vertex x="-11.2754" y="11.0334"/>
+<vertex x="-11.247353125" y="-10.5"/>
+<vertex x="11.252646875" y="-10.5"/>
+<vertex x="11.2246" y="11.0334"/>
+</polygon>
+</signal>
+<signal name="N$4">
+<polygon width="0.254" layer="16" isolate="0.381">
+<vertex x="-11.2754" y="11.0334"/>
+<vertex x="-11.247353125" y="-10.5"/>
+<vertex x="11.252646875" y="-10.5"/>
+<vertex x="11.2246" y="11.0334"/>
+</polygon>
+</signal>
