File: board_v2/Board_v2.brd (EAGLE design)
At the start: 135.1 x 89 mm, 38 parts, among them IC1 MAX7219, IC2 MAX7219, IC3 MAX7219, SW1 ROTARY SWITCH

Commit message: added board v2 files with annotations from board v1
Connections:
- removed net N$7: R4.P$2, SW1.C1
- net 3.3V: now also R4.P$2, SW1.C1
Routing:
- net N$7: track 22.7 -> 0.00 mm
- net STA: track 49.7 -> 51.6 mm
Other:
- board text added: "KETTLE META-CONTROLLER rev1. Jan-2019 Design Informatics"
