File: board_v2/Board_v2.brd (EAGLE design)
At the start: 135.1 x 89 mm, 46 parts, among them IC1 MAX7219, IC2 MAX7219, IC3 MAX7219, SW1 ROTARY SWITCH, SW2 ROTARY SWITCH

Commit message: functional version of bars_displayval.ino
Connections:
- net SEGDP1: now also IC1.22
- net SEGDP2: now also IC2.22
