File: board_v2/Board_v2.sch (EAGLE design)
At the start: 46 parts, among them IC1 MAX7219, IC2 MAX7219, IC3 MAX7219, SW1 ROTARY SWITCH, SW2 ROTARY SWITCH

Commit message: selector leds working with rotary switch
Other:
- note added: "There should not be connections to DP(decimal places) LED.. This is probably due to grid errors in 7seg symbols"
Changed lines of the file:
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@@
 see below for correct way</text>
 <text x="-469.9" y="439.42" size="1.778" layer="94">This net was not on board v1</text>
+<text x="-589.28" y="520.7" size="1.778" layer="94">There should not be connections to DP(decimal places) LED..
+This is probably due to grid errors in 7seg symbols</text>
 </plain>
 <instances>
@@
 <wire x1="-157.48" y1="121.919996875" x2="-157.48" y2="121.92" width="0.1524" layer="91"/>
 <wire x1="-157.48" y1="121.919996875" x2="-142.24" y2="121.919996875" width="0.1524" layer="91"/>
-<wire x1="-142.24" y1="121.919996875" x2="-142.24" y2="119.38" width="0.1524" layer="91"/>
 <junction x="-157.48" y="121.919996875"/>
 <label x="-149.86" y="121.92" size="1.778" layer="95"/>
@@
 <wire x1="-157.48" y1="40.639996875" x2="-157.48" y2="40.64" width="0.1524" layer="91"/>
 <wire x1="-157.48" y1="40.639996875" x2="-144.78" y2="40.639996875" width="0.1524" layer="91"/>
-<wire x1="-144.78" y1="40.639996875" x2="-144.78" y2="38.1" width="0.1524" layer="91"/>
 <junction x="-157.48" y="40.639996875"/>
 <label x="-149.86" y="40.64" size="1.778" layer="95"/>
@@
 <wire x1="-91.4908" y1="226.043065625" x2="-76.2" y2="226.043065625" width="0.1524" layer="91"/>
 <wire x1="-76.2" y1="226.043065625" x2="-76.2" y2="226.06" width="0.1524" layer="91"/>
-<label x="-78.74" y="226.06" size="1.778" layer="95"/>
+<label x="-83.82" y="226.06" size="1.778" layer="95"/>
 </segment>
 </net>
@@
 <wire x1="-91.4908" y1="248.903065625" x2="-73.66" y2="248.903065625" width="0.1524" layer="91"/>
 <wire x1="-73.66" y1="248.903065625" x2="-73.66" y2="248.92" width="0.1524" layer="91"/>
-<label x="-78.74" y="248.92" size="1.778" layer="95"/>
+<label x="-83.82" y="248.92" size="1.778" layer="95"/>
 </segment>
 </net>
@@
 <wire x1="-91.4908" y1="271.763065625" x2="-76.2" y2="271.763065625" width="0.1524" layer="91"/>
 <wire x1="-76.2" y1="271.763065625" x2="-76.2" y2="271.78" width="0.1524" layer="91"/>
-<label x="-78.74" y="271.78" size="1.778" layer="95"/>
+<label x="-83.82" y="271.78" size="1.778" layer="95"/>
 </segment>
 </net>
@@
 <wire x1="-91.4908" y1="294.623065625" x2="-91.4908" y2="294.64" width="0.1524" layer="91"/>
 <wire x1="-91.4908" y1="294.64" x2="-76.2" y2="294.64" width="0.1524" layer="91"/>
-<label x="-78.74" y="294.64" size="1.778" layer="95"/>
+<label x="-83.82" y="294.64" size="1.778" layer="95"/>
 </segment>
 </net>
@@
 <pinref part="SEV10" gate="G$1" pin="7DP"/>
 <wire x1="-157.48" y1="99.057175" x2="-144.78" y2="99.057175" width="0.1524" layer="91"/>
-<wire x1="-144.78" y1="99.057175" x2="-144.78" y2="96.52" width="0.1524" layer="91"/>
-</segment>
-</net>
+<label x="-149.86" y="99.06" size="1.778" layer="95"/>
+</segment>
+</net>

Commit message: added fade test sketch
Other:
- note removed: "There should not be connections to DP(decimal places) LED.. This is probably due to grid errors in 7seg symbols"
Changed lines of the file:
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@@
 - remove al DP connections to seven segments!
 - fix grid error on symbols
-- add top and bottom labels for clarity</text>
+- add top and bottom labels for clarity
+- There should not be connections to DP(decimal places) LED..This is probably due to grid errors in 7seg symbols
+- Rotary switch should(?) be replaced with rotary encoder</text>
 <wire x1="-480.06" y1="424.18" x2="-480.06" y2="365.76" width="0.1524" layer="94"/>
 <wire x1="-480.06" y1="365.76" x2="-525.78" y2="365.76" width="0.1524" layer="94"/>
@@
 see below for correct way</text>
 <text x="-469.9" y="439.42" size="1.778" layer="94">This net was not on board v1</text>
-<text x="-589.28" y="520.7" size="1.778" layer="94">There should not be connections to DP(decimal places) LED..
-This is probably due to grid errors in 7seg symbols</text>
 </plain>
 <instances>
