File: board_v2/Board_v2.sch (EAGLE design)
At the start: 46 parts, among them IC1 MAX7219, IC2 MAX7219, IC3 MAX7219, SW1 ROTARY SWITCH, SW2 ROTARY SWITCH

Commit message: functional version of bars_displayval.ino
Connections:
- net SEGDP1: now also IC1.SEGDP
- net SEGDP2: now also IC2.SEGDP
Other:
- note added: "Address 0"
- note added: "Address 1"
- note added: "Address 2"
Changed lines of the file:
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@@
 <wire x1="-393.7" y1="368.3" x2="-462.28" y2="368.3" width="0.1524" layer="94"/>
 <wire x1="-462.28" y1="368.3" x2="-462.28" y2="421.64" width="0.1524" layer="94"/>
-<text x="-589.28" y="601.98" size="2.54" layer="94" align="top-left">Board  v1: with review annotations
+<text x="-584.2" y="612.14" size="2.54" layer="94" align="top-left">Board  v1: with review annotations
 - convert holes to components
 - debounce buttons
@@
 - There should not be connections to DP(decimal places) LED..This is probably due to grid errors in 7seg symbols
 - Rotary switch should(?) be replaced with rotary encoder
-- add EEPROM to store karma points </text>
+- add EEPROM to store karma points
+- SEGDP nets not properly connected!
+- modify DP on MAX symbol so it sits above the other digits(because it is first in the ledcontrol library)</text>
 <wire x1="-480.06" y1="424.18" x2="-480.06" y2="365.76" width="0.1524" layer="94"/>
 <wire x1="-480.06" y1="365.76" x2="-525.78" y2="365.76" width="0.1524" layer="94"/>
@@
 see below for correct way</text>
 <text x="-469.9" y="439.42" size="1.778" layer="94">This net was not on board v1</text>
+<text x="-276.86" y="477.52" size="1.778" layer="94">Address 0</text>
+<text x="-276.86" y="350.52" size="1.778" layer="94">Address 1</text>
+<text x="-276.86" y="193.04" size="1.778" layer="94">Address 2</text>
 </plain>
 <instances>
@@
 <label x="-157.48" y="497.84" size="1.778" layer="95" rot="R90"/>
 </segment>
+<segment>
+<pinref part="IC1" gate="G$1" pin="SEGDP"/>
+<wire x1="-256.54" y1="426.72" x2="-243.84" y2="426.72" width="0.1524" layer="91"/>
+<label x="-254" y="426.72" size="1.778" layer="95"/>
+</segment>
 </net>
 <net name="SEGG1" class="0">
@@
 <label x="-157.48" y="320.04" size="1.778" layer="95" rot="R90"/>
 </segment>
-</net>
+<segment>
+<pinref part="IC2" gate="G$1" pin="SEGDP"/>
+<wire x1="-256.54" y1="304.8" x2="-241.3" y2="304.8" width="0.1524" layer="91"/>
+<label x="-254" y="304.8" size="1.778" layer="95"/>
+</segment>
+</net>
